Commit message: split rubber hand

File: G1/g1_23dof_rubber_hand.urdf (robot description, URDF)
Before this commit: robot g1_23dof_rev_1_0, 31 links, 30 joints
Links:
- removed link left_wrist_roll_rubber_hand
- removed link right_wrist_roll_rubber_hand
- added link left_rubber_hand_link, mass 0.1; collision mesh filename=meshes/left_rubber_hand.STL; visual mesh filename=meshes/left_rubber_hand.STL
- added link left_wrist_roll_link, mass 0.35692864; collision mesh filename=meshes/left_wrist_roll.STL; visual mesh filename=meshes/left_wrist_roll.STL
- added link right_rubber_hand_link, mass 0.1; collision mesh filename=meshes/right_rubber_hand.STL; visual mesh filename=meshes/right_rubber_hand.STL
- added link right_wrist_roll_link, mass 0.35692864; collision mesh filename=meshes/right_wrist_roll.STL; visual mesh filename=meshes/right_wrist_roll.STL
Joints:
- added joint left_rubber_hand_joint: type fixed, parent left_wrist_roll_link, child left_rubber_hand_link, origin xyz=0.121 0.0055 0.0015 rpy=0 0 0
- added joint right_rubber_hand_joint: type fixed, parent right_wrist_roll_link, child right_rubber_hand_link, origin xyz=0.121 -0.0055 0.0015 rpy=0 0 0
- joint left_wrist_roll_joint: child left_wrist_roll_rubber_hand -> left_wrist_roll_link
- joint right_wrist_roll_joint: child right_wrist_roll_rubber_hand -> right_wrist_roll_link

Commit message: add usd

File: G1/g1_23dof_rubber_hand.urdf (robot description, URDF)
Before this commit: robot g1_23dof_rev_1_0, 33 links, 32 joints
Links:
- removed link left_rubber_hand_link
- removed link right_rubber_hand_link
- added link left_rubber_hand, mass 0.1; collision mesh filename=meshes/left_rubber_hand.STL; visual mesh filename=meshes/left_rubber_hand.STL
- added link right_rubber_hand, mass 0.1; collision mesh filename=meshes/right_rubber_hand.STL; visual mesh filename=meshes/right_rubber_hand.STL
Joints:
- joint left_rubber_hand_joint: child left_rubber_hand_link -> left_rubber_hand
- joint right_rubber_hand_joint: child right_rubber_hand_link -> right_rubber_hand
